Commit message: add rs urdf parse

File: urdf/00-arm-rs_asm-v3/urdf/00-arm-rs_asm-v3.urdf (robot description, URDF)
Before this commit: robot 00-arm-rs_asm-v3, 10 links, 9 joints
Links:
- link gripper_end: geometry collision mesh filename=meshes/gripper_end.STL; visual mesh filename=meshes/gripper_end.STL
- link gripper_left: geometry collision mesh filename=meshes/gripper_left.STL; visual mesh filename=meshes/gripper_left.STL
- link gripper_right: geometry collision mesh filename=meshes/gripper_right.STL; visual mesh filename=meshes/gripper_right.STL
- link link2: geometry collision mesh filename=meshes/link2.STL; visual mesh filename=meshes/cnc2.STL
- link link3: geometry collision mesh filename=meshes/link3.STL; visual mesh filename=meshes/link3.STL
- link link4: geometry collision mesh filename=meshes/link4.STL; visual mesh filename=meshes/link4.STL
- link link5: geometry collision mesh filename=meshes/link5.STL; visual mesh filename=meshes/link5.STL

Commit message: finish gravity

File: urdf/00-arm-rs_asm-v3/urdf/00-arm-rs_asm-v3.urdf (robot description, URDF)
Before this commit: robot 00-arm-rs_asm-v3, 10 links, 9 joints
Joints:
- removed joint j_gripper_end
- removed joint joint_left
- removed joint joint_right
- added joint gripper_joint: type fixed, parent link6, child gripper_end, origin xyz=0 0 0.16621 rpy=3.1416 -1.5708 0, axis 0 0 0
- added joint gripper_joint_left: type prismatic, parent gripper_end, child gripper_left, origin xyz=-0.041939 -7.3385E-05 0 rpy=1.5708 -1.5708 0, axis 0 0 1, limit lower=0 upper=0.05 effort=500 velocity=10
- added joint gripper_joint_right: type prismatic, parent gripper_end, child gripper_right, origin xyz=-0.041939 7.3385E-05 0 rpy=-1.5708 -1.5708 0, axis 0 0 1, limit lower=0 upper=0.0715 effort=500 velocity=10
